File: Wireless Split/Wireless Split.kicad_sch (KiCad schematic)
At the start: 0 parts

Commit message: final
Parts:
- added BO1, BO2, BO3: Break off, Mousebites:mouse-bite-5mm-slot, symbol Mechanical:MountingHole
- added H1, H2, H3, H4, H5, H6, H7, H8: MountingHole, MountingHole:MountingHole_2.2mm_M2, symbol Mechanical:MountingHole
Other:
- added sheet Left (Half.kicad_sch)
- added sheet Right (Half.kicad_sch)
